File: digital_in.sch (KiCad schematic (older format))
At the start: 24 parts

Commit message: added missing component values working on BOM
Parts:
- C23, C24, C25, C26, C27, C28: Mouser (none) -> 80-C0805C105M4R
- D12, D13, D14, D15, D16, D17: Mouser (none) -> 863-BAT54SLT1G
Changed lines of the file:
@@
 F 2 "Capacitor_SMD:C_0805_2012Metric" H 3588 2150 50  0001 C CNN
 F 3 "~" H 3550 2300 50  0001 C CNN
+F 4 "80-C0805C105M4R " H 3550 2300 50  0001 C CNN "Mouser"
 	1    3550 2300
 	1    0    0    -1
@@
 F 2 "Capacitor_SMD:C_0805_2012Metric" H 3588 4150 50  0001 C CNN
 F 3 "~" H 3550 4300 50  0001 C CNN
+F 4 "80-C0805C105M4R " H 3550 4300 50  0001 C CNN "Mouser"
 	1    3550 4300
 	1    0    0    -1
@@
 F 2 "Capacitor_SMD:C_0805_2012Metric" H 3588 6250 50  0001 C CNN
 F 3 "~" H 3550 6400 50  0001 C CNN
+F 4 "80-C0805C105M4R " H 3550 6400 50  0001 C CNN "Mouser"
 	1    3550 6400
 	1    0    0    -1
@@
 F 2 "Capacitor_SMD:C_0805_2012Metric" H 7588 2150 50  0001 C CNN
 F 3 "~" H 7550 2300 50  0001 C CNN
+F 4 "80-C0805C105M4R " H 7550 2300 50  0001 C CNN "Mouser"
 	1    7550 2300
 	1    0    0    -1
@@
 F 2 "Capacitor_SMD:C_0805_2012Metric" H 7588 4150 50  0001 C CNN
 F 3 "~" H 7550 4300 50  0001 C CNN
+F 4 "80-C0805C105M4R " H 7550 4300 50  0001 C CNN "Mouser"
 	1    7550 4300
 	1    0    0    -1
@@
 F 2 "Capacitor_SMD:C_0805_2012Metric" H 7588 6250 50  0001 C CNN
 F 3 "~" H 7550 6400 50  0001 C CNN
+F 4 "80-C0805C105M4R " H 7550 6400 50  0001 C CNN "Mouser"
 	1    7550 6400
 	1    0    0    -1
@@
 F 2 "Package_TO_SOT_SMD:SOT-23" H 3075 2175 50  0001 L CNN
 F 3 "https://www.diodes.com/assets/Datasheets/ds11005.pdf" H 2880 2050 50  0001 C CNN
+F 4 "863-BAT54SLT1G" H 3000 2050 50  0001 C CNN "Mouser"
 	1    3000 2050
 	0    -1   -1   0
@@
 F 2 "Package_TO_SOT_SMD:SOT-23" H 3075 4175 50  0001 L CNN
 F 3 "https://www.diodes.com/assets/Datasheets/ds11005.pdf" H 2880 4050 50  0001 C CNN
+F 4 "863-BAT54SLT1G" H 3000 4050 50  0001 C CNN "Mouser"
 	1    3000 4050
 	0    -1   -1   0
@@
 F 2 "Package_TO_SOT_SMD:SOT-23" H 3075 6275 50  0001 L CNN
 F 3 "https://www.diodes.com/assets/Datasheets/ds11005.pdf" H 2880 6150 50  0001 C CNN
+F 4 "863-BAT54SLT1G" H 3000 6150 50  0001 C CNN "Mouser"
 	1    3000 6150
 	0    -1   -1   0
@@
 F 2 "Package_TO_SOT_SMD:SOT-23" H 7075 2175 50  0001 L CNN
 F 3 "https://www.diodes.com/assets/Datasheets/ds11005.pdf" H 6880 2050 50  0001 C CNN
+F 4 "863-BAT54SLT1G" H 7000 2050 50  0001 C CNN "Mouser"
 	1    7000 2050
 	0    -1   -1   0
@@
 F 2 "Package_TO_SOT_SMD:SOT-23" H 7075 4175 50  0001 L CNN
 F 3 "https://www.diodes.com/assets/Datasheets/ds11005.pdf" H 6880 4050 50  0001 C CNN
+F 4 "863-BAT54SLT1G" H 7000 4050 50  0001 C CNN "Mouser"
 	1    7000 4050
 	0    -1   -1   0
@@
 F 2 "Package_TO_SOT_SMD:SOT-23" H 7075 6275 50  0001 L CNN
 F 3 "https://www.diodes.com/assets/Datasheets/ds11005.pdf" H 6880 6150 50  0001 C CNN
+F 4 "863-BAT54SLT1G" H 7000 6150 50  0001 C CNN "Mouser"
 	1    7000 6150
 	0    -1   -1   0

Commit message: cleaned BOMs
Parts:
- R42, R43, R44, R48, R49, R50: Mouser (none) -> 279-CRGCQ0805F10K
- R45, R46, R47, R51, R52, R53: Mouser (none) -> 279-CRGCQ0805F100K
Changed lines of the file:
@@
 F 2 "Resistor_SMD:R_0805_2012Metric" V 2030 2050 50  0001 C CNN
 F 3 "~" H 2100 2050 50  0001 C CNN
+F 4 "279-CRGCQ0805F10K" H 2100 2050 50  0001 C CNN "Mouser"
 	1    2100 2050
 	0    1    1    0
@@
 F 2 "Resistor_SMD:R_0805_2012Metric" V 2480 2350 50  0001 C CNN
 F 3 "~" H 2550 2350 50  0001 C CNN
+F 4 "279-CRGCQ0805F100K" H 2550 2350 50  0001 C CNN "Mouser"
 	1    2550 2350
 	-1   0    0    1
@@
 F 2 "Resistor_SMD:R_0805_2012Metric" V 2030 4050 50  0001 C CNN
 F 3 "~" H 2100 4050 50  0001 C CNN
+F 4 "279-CRGCQ0805F10K" H 2100 4050 50  0001 C CNN "Mouser"
 	1    2100 4050
 	0    1    1    0
@@
 F 2 "Resistor_SMD:R_0805_2012Metric" V 2480 4350 50  0001 C CNN
 F 3 "~" H 2550 4350 50  0001 C CNN
+F 4 "279-CRGCQ0805F100K" H 2550 4350 50  0001 C CNN "Mouser"
 	1    2550 4350
 	-1   0    0    1
@@
 F 2 "Resistor_SMD:R_0805_2012Metric" V 2030 6150 50  0001 C CNN
 F 3 "~" H 2100 6150 50  0001 C CNN
+F 4 "279-CRGCQ0805F10K" H 2100 6150 50  0001 C CNN "Mouser"
 	1    2100 6150
 	0    1    1    0
@@
 F 2 "Resistor_SMD:R_0805_2012Metric" V 2480 6450 50  0001 C CNN
 F 3 "~" H 2550 6450 50  0001 C CNN
+F 4 "279-CRGCQ0805F100K" H 2550 6450 50  0001 C CNN "Mouser"
 	1    2550 6450
 	-1   0    0    1
@@
 F 2 "Resistor_SMD:R_0805_2012Metric" V 6030 2050 50  0001 C CNN
 F 3 "~" H 6100 2050 50  0001 C CNN
+F 4 "279-CRGCQ0805F10K" H 6100 2050 50  0001 C CNN "Mouser"
 	1    6100 2050
 	0    1    1    0
@@
 F 2 "Resistor_SMD:R_0805_2012Metric" V 6480 2350 50  0001 C CNN
 F 3 "~" H 6550 2350 50  0001 C CNN
+F 4 "279-CRGCQ0805F100K" H 6550 2350 50  0001 C CNN "Mouser"
 	1    6550 2350
 	-1   0    0    1
@@
 F 2 "Resistor_SMD:R_0805_2012Metric" V 6030 4050 50  0001 C CNN
 F 3 "~" H 6100 4050 50  0001 C CNN
+F 4 "279-CRGCQ0805F10K" H 6100 4050 50  0001 C CNN "Mouser"
 	1    6100 4050
 	0    1    1    0
@@
 F 2 "Resistor_SMD:R_0805_2012Metric" V 6480 4350 50  0001 C CNN
 F 3 "~" H 6550 4350 50  0001 C CNN
+F 4 "279-CRGCQ0805F100K" H 6550 4350 50  0001 C CNN "Mouser"
 	1    6550 4350
 	-1   0    0    1
@@
 F 2 "Resistor_SMD:R_0805_2012Metric" V 6030 6150 50  0001 C CNN
 F 3 "~" H 6100 6150 50  0001 C CNN
+F 4 "279-CRGCQ0805F10K" H 6100 6150 50  0001 C CNN "Mouser"
 	1    6100 6150
 	0    1    1    0
@@
 F 2 "Resistor_SMD:R_0805_2012Metric" V 6480 6450 50  0001 C CNN
 F 3 "~" H 6550 6450 50  0001 C CNN
+F 4 "279-CRGCQ0805F100K" H 6550 6450 50  0001 C CNN "Mouser"
 	1    6550 6450
 	-1   0    0    1
